Commit message: update moveto irl

File: ros_ws/src/moveto/urdf/team2_robot.urdf (robot description, URDF)
Before this commit: robot myrobot, 8 links, 7 joints
Links:
- link link2: geometry visual box size=0.00635 0.3048 0.045
- link link3: geometry visual box size=0.00635 0.3048 0.045
Joints:
- joint motor3_attachment: origin xyz=0 0.2032 0 rpy=0 0 0 -> xyz=0 0.3048 0 rpy=0 0 0

File: ros_ws/src/myrobot/urdf/team2_robot.urdf (robot description, URDF)
Before this commit: robot myrobot, 8 links, 7 joints
Links:
- link link2: geometry visual box size=0.00635 0.2042 0.045
- link link3: geometry visual box size=0.00635 0.2042 0.045
Joints:
- joint motor3_attachment: origin xyz=0 0.2032 0 rpy=0 0 0 -> xyz=0 0.2042 0 rpy=0 0 0
